Commit message: latest

File: sodabot.urdf.xacro (robot description, xacro)
@@ -110,5 +110,5 @@
 		<inertial>
 			<!--
-				From meshlab:
+				From meshlab: (old)
 				LOG: 2 Mesh Bounding Box Size 35.699898 41.299900 66.638039
 				LOG: 2 Mesh Bounding Box Diag 86.144028
@@ -127,7 +127,24 @@
 				LOG: 2 axis momenta are :
 				LOG: 2     | 1425298.500000  1363803.125000  366547.718750 |
+				(new)
+				LOG: 2 Mesh Bounding Box Size 35.699898 41.299900 66.638039
+				LOG: 2 Mesh Bounding Box Diag 86.144028
+				LOG: 2 Mesh Volume  is 1295.270142
+				LOG: 2 Mesh Surface is 9440.942383
+				LOG: 2 Thin shell barycenter  -11.234900  -0.000052  41.190914
+				LOG: 2 Center of Mass  is -11.913177 -0.000048 40.919144
+				LOG: 2 Inertia Tensor is :
+				LOG: 2     | 1423924.500000   0.409780  -38116.269531 |
+				LOG: 2     |  0.409780  1363803.125000  -0.002875 |
+				LOG: 2     | -38116.269531  -0.002875  367921.718750 |
+				LOG: 2 Principal axes are :
+				LOG: 2     |  0.999351  -0.000007   0.036025 |
+				LOG: 2     |  0.000007   1.000000  -0.000000 |
+				LOG: 2     | -0.036025   0.000000   0.999351 |
+				LOG: 2 axis momenta are :
+				LOG: 2     | 1425298.500000  1363803.125000  366547.718750 |
 			-->
 			<origin
-				xyz="${11.913177/scaling} ${0/scaling} ${40.919144/scaling}"
+				xyz="${-11.913177/scaling} ${0/scaling} ${41.190914/scaling}"
 				rpy="0 0 0"/>
 			<mass
@@ -135,6 +152,6 @@
 <!--			<xacro:cuboid_inertia mass="${chassis_mass}" sx="${bottomPlateDepth}" sy="${baseWidth}" sz="${topPlateElevation-bottomPlateElevation}"/> -->
 			<inertia
-				ixx="${1423924.500000*inertial_scale}"	ixy="${0.409780*inertial_scale}"			ixz="${38116.269531*inertial_scale}"
-														iyy="${1363803.125000*inertial_scale}"		iyz="${0.002875*inertial_scale}"
+				ixx="${1423924.500000*inertial_scale}"	ixy="${0.409780*inertial_scale}"			ixz="${-38116.269531*inertial_scale}"
+														iyy="${1363803.125000*inertial_scale}"		iyz="${-0.002875*inertial_scale}"
 																									izz="${367921.718750*inertial_scale}"
 				/>
@@ -249,5 +266,5 @@
 	  <parent link="base_link"/>
 	  <child link="mwheel"/>
-	  <origin rpy="0 0 0" xyz="${bottomPlateDepth-wheelsAtDepth-0.01} 0 ${bottomPlateElevation - 0.06}"/>
+	  <origin rpy="0 0 0" xyz="${-bottomPlateDepth+wheelsAtDepth+0.01} 0 ${bottomPlateElevation - 0.06}"/>
 	  <dynamics damping="0.0" friction="0.0"/>
 	</joint>
@@ -454,5 +471,5 @@
 	  <parent link="base_link"/>
 	  <child link="head_pan_base"/>
-	  <origin rpy="0 0 0" xyz="0.090 0 ${topPlateElevation + plateThickness + 0.0466/2}"/>
+	  <origin rpy="0 0 0" xyz="0 0 ${topPlateElevation + plateThickness + 0.0466/2}"/>
 	  <dynamics damping="0.0" friction="0.0"/>
 	</joint>
@@ -476,5 +493,5 @@
 	  <parent link="head_pan_base"/>
 	  <child link="head_tilt_base"/>
-	  <origin rpy="0 0 0" xyz="0 0 ${0.0466}"/>
+	  <origin rpy="0 0 0" xyz="0 0 ${0.065}"/>
 	  <limit lower="${-pi/2}" upper="${pi/2}" effort="1" velocity="${pi/4}"/>
 	  <dynamics damping="1.0" friction="1.0"/>

Commit message: latest

File: sodabot.urdf.xacro (robot description, xacro)
@@ -373,6 +373,8 @@
     <link name="${name}_kinect2_link">
 	  <xacro:cuboid_inertial mass="0.0001" sx="0.065" sy="0.250" sz="0.050"/>
+<!--
+      <origin xyz="0 0 0" rpy="0 0.026179929 0"/>
+-->
       <visual>
-        <origin xyz="0 0 0" rpy="0 0 0"/>
         <geometry>
 	   		<box size="0.065 0.250 0.050"/>
@@ -383,5 +385,4 @@
       </visual>
       <collision>
-        <origin xyz="0 0 0" rpy="0 0 0"/>
         <geometry>
 	   		<box size="0.065 0.250 0.050"/>
@@ -391,5 +392,8 @@
     <!-- kinect2 ir sensor physical attachment -->
     <joint name="${name}_kinect2_ir_joint" type="fixed">
+		  <!--
       <origin xyz="-0.032267 -0.0475 0.155" rpy="0 0 0"/>
+			-->
+      <origin xyz="0 -0.0475 0" rpy="0 0 0"/>
       <parent link="${name}_kinect2_link"/>
       <child link="${name}_kinect2_ir_link"/>
@@ -466,10 +470,10 @@
 	  		<origin rpy="0 0 0" xyz="0 0 0"/>
 		</collision>
-		<xacro:cuboid_inertial mass="0.94" sx="0.06352" sy="0.02975" sz="0.0466"/>
+		<xacro:cuboid_inertial mass="0.94" sx="0.06352" sy="0.02975" sz="0.0566"/>
 	</link>
     <joint name="base_to_head_pan_base_joint" type="fixed">
 	  <parent link="base_link"/>
 	  <child link="head_pan_base"/>
-	  <origin rpy="0 0 0" xyz="0 0 ${topPlateElevation + plateThickness + 0.0466/2}"/>
+	  <origin rpy="0 0 0" xyz="0 0 ${topPlateElevation + plateThickness + 0.0566/2}"/>
 	  <dynamics damping="0.0" friction="0.0"/>
 	</joint>
@@ -493,5 +497,5 @@
 	  <parent link="head_pan_base"/>
 	  <child link="head_tilt_base"/>
-	  <origin rpy="0 0 0" xyz="0 0 ${0.065}"/>
+	  <origin rpy="0 0 0" xyz="0 0 ${0.0687}"/>
 	  <limit lower="${-pi/2}" upper="${pi/2}" effort="1" velocity="${pi/4}"/>
 	  <dynamics damping="1.0" friction="1.0"/>
@@ -515,10 +519,10 @@
 	  <parent link="head_tilt_base"/>
 	  <child link="head_kinect_mount_link"/>
-	  <origin rpy="0 0 0" xyz="0 0 0"/>
+	  <origin rpy="0 0 0" xyz="-0.01 0 0"/>
 	  <limit lower="${-pi*0.4}" upper="${pi*0.4}" effort="1" velocity="${pi/4}"/>
 	  <dynamics damping="1.0" friction="1.0"/>
 	</joint>
     <xacro:kinect2_v0 name="head_mount" parent="head_kinect_mount_link" >
-      <origin xyz="0 0 ${0.080 - 0.050/2}" rpy="0 0 0" />
+      <origin xyz="0.01 -0.015 ${0.075}" rpy="0 0.046179929 0" />
     </xacro:kinect2_v0>
 <!--
@@ -634,4 +638,5 @@
 			<odometryTopic>odom</odometryTopic>
 		</plugin>
+		80 - 0.050/2
 	</gazebo>
 </robot>

Commit message: latest

File: sodabot.urdf.xacro (robot description, xacro)
@@ -248,5 +248,5 @@
 	  <parent link="base_link"/>
 	  <child link="rwheel"/>
-	  <origin rpy="${-pi/2} 0 0" xyz="0 ${-baseWidth/2 -wheelOffsetFromBase} ${bottomPlateElevation - wheelJointHeightFromBase}"/>
+	  <origin rpy="${pi/2} 0 0" xyz="0 ${baseWidth/2  + wheelOffsetFromBase} ${bottomPlateElevation - wheelJointHeightFromBase}"/>
 	  <dynamics damping="0.0" friction="0.0"/>
 	  <limit effort="100" velocity="100"/>
@@ -257,5 +257,5 @@
 	  <parent link="base_link"/>
 	  <child link="lwheel"/>
-	  <origin rpy="${pi/2} 0 0" xyz="0 ${baseWidth/2 + wheelOffsetFromBase} ${bottomPlateElevation - wheelJointHeightFromBase}"/>
+	  <origin rpy="${-pi/2} 0 0" xyz="0 ${-baseWidth/2 - wheelOffsetFromBase} ${bottomPlateElevation - wheelJointHeightFromBase}"/>
 	  <dynamics damping="0.0" friction="0.0"/>
 	  <limit effort="100" velocity="100"/>
